File: ice60.kicad_pcb (KiCad board)
At the start: 2 copper layers, 284.8 x 94.2 mm, 199 parts, among them J1 SWD, J2 JST SH 4-pin, SW0 SW_Push, SW1 MX_SW_solder, SW10 MX_SW_solder, SW11 MX_SW_solder, SW12 MX_SW_solder, SW13 MX_SW_solder, SW14 MX_SW_solder, SW15 MX_SW_solder, SW16 MX_SW_solder, SW17 MX_SW_solder, SW18 MX_SW_solder, SW19 MX_SW_solder, SW2 MX_SW_solder, SW20 MX_SW_solder, SW21 MX_SW_solder, SW22 MX_SW_solder, SW23 MX_SW_solder, SW24 MX_SW_solder, SW25 MX_SW_solder, SW26 MX_SW_solder, SW27 MX_SW_solder, SW28 MX_SW_solder, SW29 MX_SW_solder, SW3 MX_SW_solder, SW30 MX_SW_solder, SW31 MX_SW_solder, SW32 MX_SW_solder, SW33 MX_SW_solder, SW34 MX_SW_solder, SW35 MX_SW_solder, SW36 MX_SW_solder, SW37 MX_SW_solder, SW38 MX_SW_solder, SW39 MX_SW_solder, SW4 MX_SW_solder, SW40 MX_SW_solder, SW41 MX_SW_solder, SW42 MX_SW_solder, SW43 MX_SW_solder, SW44 MX_SW_solder, SW45 MX_SW_solder, SW46 MX_SW_solder, SW47 MX_SW_solder, SW48 MX_SW_solder, SW49 MX_SW_solder, SW5 MX_SW_solder, SW50 MX_SW_solder, SW51 MX_SW_solder, SW52 MX_SW_solder, SW53 MX_SW_solder, SW54 MX_SW_solder, SW55 MX_SW_solder, SW56 MX_SW_solder, SW57 MX_SW_solder, SW58 MX_SW_solder, SW59 MX_SW_solder, SW6 MX_SW_solder, SW60 MX_SW_solder, SW61 MX_SW_solder, SW62 MX_SW_solder, SW63 MX_SW_solder, SW64 MX_SW_solder, SW65 MX_SW_solder, SW66 MX_SW_solder, SW67 MX_SW_solder, SW68 MX_SW_solder, SW69 MX_SW_solder, SW7 MX_SW_solder, SW70 MX_SW_solder, SW71 MX_SW_solder, SW72 MX_SW_solder, SW73 MX_SW_solder, SW74 MX_SW_solder, SW75 MX_SW_solder, SW76 MX_SW_solder, SW77 MX_SW_solder, SW78 MX_SW_solder, SW79 MX_SW_solder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

Commit message: delete sneaky track tails
Routing:
- net Net-(D61-Pad2): track 30.2 -> 28.3 mm
- net COL08: track 269.9 -> 268.7 mm
- net Net-(D44-Pad2): track 12.4 -> 11.6 mm
- net Net-(D28-Pad2): track 27.6 -> 27.0 mm
- net Net-(D63-Pad2): track 8.14 -> 7.56 mm
Changed lines of the file:
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@@
   (segment (start 56.299233 73.364858) (end 55.959375 73.704716) (width 0.2) (layer "B.Cu") (net 6))
   (segment (start 62.652499 63.287499) (end 61.595 62.23) (width 0.2) (layer "B.Cu") (net 6))
-  (segment (start 56.220177 73.443915) (end 56.299233 73.364858) (width 0.2) (layer "B.Cu") (net 6))
   (segment (start 67.865625 62.3925) (end 67.155 62.3925) (width 0.3) (layer "B.Cu") (net 6))
   (segment (start 66.935802 63.322323) (end 67.865625 62.3925) (width 0.2) (layer "B.Cu") (net 6))
@@
   (segment (start 301.002651 56.130776) (end 301.002651 55.88) (width 0.3) (layer "F.Cu") (net 35))
   (segment (start 301.625 56.753125) (end 301.002651 56.130776) (width 0.3) (layer "F.Cu") (net 35))
-  (segment (start 303.05375 65.405) (end 303.133125 65.405) (width 0.3) (layer "F.Cu") (net 35))
-  (segment (start 303.133125 65.405) (end 303.2125 65.484375) (width 0.3) (layer "F.Cu") (net 35))
   (segment (start 301.625 63.97625) (end 301.625 56.753125) (width 0.3) (layer "F.Cu") (net 35))
   (segment (start 303.05375 65.405) (end 301.625 63.97625) (width 0.3) (layer "F.Cu") (net 35))
   (segment (start 296.2275 52.3875) (end 299.640625 52.3875) (width 0.3) (layer "B.Cu") (net 35))
   (segment (start 289.004375 56.895) (end 289.004375 56.8325) (width 0.3) (layer "B.Cu") (net 35))
-  (segment (start 301.002651 55.88) (end 301.3075 56.184849) (width 0.3) (layer "B.Cu") (net 35))
   (segment (start 289.004375 56.8325) (end 291.7825 56.8325) (width 0.3) (layer "B.Cu") (net 35))
   (segment (start 299.640625 52.3875) (end 301.002651 53.749526) (width 0.3) (layer "B.Cu") (net 35))
@@
   (segment (start 287.9725 72.786875) (end 287.9725 72.39) (width 0.3) (layer "B.Cu") (net 47))
   (segment (start 283.765625 73.81875) (end 286.940625 73.81875) (width 0.3) (layer "B.Cu") (net 47))
-  (segment (start 287.81375 72.23125) (end 287.9725 72.39) (width 0.3) (layer "B.Cu") (net 47))
   (segment (start 278.209375 71.896875) (end 281.84375 71.896875) (width 0.3) (layer "B.Cu") (net 47))
   (segment (start 287.9725 72.39) (end 299.87875 72.39) (width 0.3) (layer "B.Cu") (net 47))
@@
   (segment (start 41.11625 93.98) (end 50.64125 93.98) (width 0.3) (layer "B.Cu") (net 49))
   (segment (start 37.7825 90.64625) (end 41.11625 93.98) (width 0.3) (layer "B.Cu") (net 49))
-  (segment (start 63.12 93.4075) (end 62.5475 93.98) (width 0.3) (layer "B.Cu") (net 50))
   (segment (start 73.50125 92.534375) (end 72.055625 93.98) (width 0.3) (layer "B.Cu") (net 50))
   (segment (start 72.055625 93.98) (end 62.5475 93.98) (width 0.3) (layer "B.Cu") (net 50))
@@
   (segment (start 297.33875 101.5375) (end 290.195 101.5375) (width 0.3) (layer "B.Cu") (net 67))
   (segment (start 242.57 104.8375) (end 242.57 105.88625) (width 0.3) (layer "B.Cu") (net 68))
-  (segment (start 238.38 110.07625) (end 237.96625 110.49) (width 0.3) (layer "B.Cu") (net 68))
   (segment (start 242.57 105.88625) (end 237.96625 110.49) (width 0.3) (layer "B.Cu") (net 68))
   (segment (start 290.195 105.88625) (end 285.59125 110.49) (width 0.3) (layer "B.Cu") (net 69))
@@
   (segment (start 201.215625 70.723125) (end 205.4225 74.93) (width 0.3) (layer "F.Cu") (net 91))
   (segment (start 206.062501 102.081251) (end 213.603126 102.081251) (width 0.3) (layer "F.Cu") (net 91))
-  (segment (start 205.978125 113.585625) (end 205.4225 113.03) (width 0.3) (layer "F.Cu") (net 91))
-  (segment (start 216.535 110.49) (end 216.535 110.96625) (width 0.3) (layer "F.Cu") (net 91))
   (segment (start 205.4225 113.03) (end 205.4225 112.87125) (width 0.3) (layer "F.Cu") (net 91))
   (segment (start 213.603126 102.081251) (end 216.535 105.013125) (width 0.3) (layer "F.Cu") (net 91))
@@
   (segment (start 116.36375 92.534375) (end 118.251875 92.534375) (width 0.3) (layer "B.Cu") (net 117))
   (segment (start 118.251875 92.534375) (end 119.6975 93.98) (width 0.3) (layer "B.Cu") (net 117))
-  (segment (start 160.17875 112.0775) (end 160.17875 113.03) (width 0.3) (layer "F.Cu") (net 118))
-  (segment (start 172.085 112.0775) (end 172.085 113.03) (width 0.3) (layer "F.Cu") (net 118))
   (segment (start 171.1325 110.07625) (end 173.25875 110.07625) (width 0.3) (layer "B.Cu") (net 118))
   (segment (start 171.1325 104.8375) (end 171.1325 107.870625) (width 0.3) (layer "B.Cu") (net 118))

Commit message: o ring mounting cutouts
Parts:
- removed the REF** at (209.2, 115.6)
- removed the REF** at (137.8, 115.6)
- removed the SW76 at (171.1, 115.6)
- removed the SW79 at (209.2, 115.6)
- renumbered SW77 to SW76, SW78 to SW77, SW80 to SW78, SW81 to SW79, SW82 to SW80, SW83 to SW81, SW84 to SW82, SW85 to SW83, SW86 to SW84, SW87 to SW85, SW88 to SW86
Connections:
- SW77 pad 1: Net-(D62-Pad2) -> COL08
- SW77 pad 2: COL08 -> Net-(D62-Pad2)
Routing:
- net COL08: track 268.7 -> 253.5 mm
- net COL05: track 199.4 -> 188.9 mm
- net COL11: track 318.6 -> 308.3 mm
- net COL12: track 357.8 -> 351.6 mm
- net Net-(D61-Pad2): track 28.3 -> 23.5 mm
- net Net-(D62-Pad2): track 26.4 -> 22.2 mm
- net COL06: track 223.6 -> 219.9 mm
- net ROW0: track 296.5 -> 294.9 mm
Other:
- board size 284.8 x 94.2 mm -> 284.7 x 94.2 mm

Commit message: tweaks
Parts:
- moved D43 14.7 mm to (52.5, 88.6)
- moved D42 9.92 mm to (305.7, 46.5)
Routing:
- net Net-(D42-Pad2): track 13.0 -> 16.2 mm
- net ROW3: track 314.4 -> 312.3 mm
- net GND: track 36.6 -> 37.7 mm
- net Net-(D60-Pad2): track 20.5 -> 21.1 mm
