File: matrix.kicad_sch (KiCad schematic)
At the start: 154 parts, among them SW1 MX_SW_solder, SW10 MX_SW_solder, SW11 MX_SW_solder, SW12 MX_SW_solder, SW13 MX_SW_solder, SW14 MX_SW_solder, SW15 MX_SW_solder, SW16 MX_SW_solder, SW17 MX_SW_solder, SW18 MX_SW_solder, SW19 MX_SW_solder, SW2 MX_SW_solder, SW20 MX_SW_solder, SW21 MX_SW_solder, SW22 MX_SW_solder, SW23 MX_SW_solder, SW24 MX_SW_solder, SW25 MX_SW_solder, SW26 MX_SW_solder, SW27 MX_SW_solder, SW28 MX_SW_solder, SW29 MX_SW_solder, SW3 MX_SW_solder, SW30 MX_SW_solder, SW31 MX_SW_solder, SW32 MX_SW_solder, SW33 MX_SW_solder, SW34 MX_SW_solder, SW35 MX_SW_solder, SW36 MX_SW_solder, SW37 MX_SW_solder, SW38 MX_SW_solder, SW39 MX_SW_solder, SW4 MX_SW_solder, SW40 MX_SW_solder, SW41 MX_SW_solder, SW42 MX_SW_solder, SW43 MX_SW_solder, SW44 MX_SW_solder, SW45 MX_SW_solder, SW46 MX_SW_solder, SW47 MX_SW_solder, SW48 MX_SW_solder, SW49 MX_SW_solder, SW5 MX_SW_solder, SW50 MX_SW_solder, SW51 MX_SW_solder, SW52 MX_SW_solder, SW53 MX_SW_solder, SW54 MX_SW_solder, SW55 MX_SW_solder, SW56 MX_SW_solder, SW57 MX_SW_solder, SW58 MX_SW_solder, SW59 MX_SW_solder, SW6 MX_SW_solder, SW60 MX_SW_solder, SW61 MX_SW_solder, SW62 MX_SW_solder, SW63 MX_SW_solder, SW64 MX_SW_solder, SW65 MX_SW_solder, SW66 MX_SW_solder, SW67 MX_SW_solder, SW68 MX_SW_solder, SW69 MX_SW_solder, SW7 MX_SW_solder, SW70 MX_SW_solder, SW71 MX_SW_solder, SW72 MX_SW_solder, SW73 MX_SW_solder, SW74 MX_SW_solder, SW75 MX_SW_solder, SW76 MX_SW_solder, SW77 MX_SW_solder, SW78 MX_SW_solder, SW79 MX_SW_solder, SW8 MX_SW_solder, SW80 MX_SW_solder, SW81 MX_SW_solder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

Commit message: tweak diodes
Connections:
- net COL00: now also SW31.2, SW32.2, SW47.2, SW48.2; no longer SW31.1, SW32.1, SW47.1, SW48.1
- net COL10: now also SW80.1; no longer SW80.2
- net COL12: now also SW28.2, SW60.2, SW61.2; no longer SW28.1, SW60.1, SW61.1
- net COL13: now also SW14.2, SW15.2, SW29.2, SW30.2, SW62.2, SW87.2, SW88.2; no longer SW14.1, SW15.1, SW29.1, SW30.1, SW62.1, SW87.1, SW88.1
- net at D80.2 (A): now also SW80.2; no longer SW80.1
- net at D62.2 (A): now also SW62.1; no longer SW62.2
- net at D28.2 (A): now also SW28.1; no longer SW28.2
- new net: D32.2 (A), SW31.1, SW32.1
- new net: D60.2 (A), SW60.1, SW61.1
- new net: D29.2 (A), SW29.1, SW30.1
- new net: D87.2 (A), SW87.1, SW88.1
- new net: D14.2 (A), SW14.1, SW15.1
- new net: D48.2 (A), SW47.1, SW48.1
Other:
- moved on the sheet: SW14, SW15, SW28, SW29, SW30, SW32, SW48, SW60, SW61, SW62, SW80, SW87
Changed lines of the file:
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@@
     (pin "2")
   )
-  (symbol (lib_id "marbastlib-mx:MX_SW_solder") (at 43.18 78.74 0) (unit 1)
-    (in_bom yes) (on_board yes)
-    (property "Reference" "SW32" (id 0) (at 43.18 71.12 0))
-    (property "Value" "MX_SW_solder" (id 1) (at 41.91 73.66 0))
+  (symbol (lib_id "marbastlib-mx:MX_SW_solder") (at 43.18 78.74 180) (unit 1)
+    (in_bom yes) (on_board yes)
+    (property "Reference" "SW32" (id 0) (at 43.18 86.36 0))
+    (property "Value" "MX_SW_solder" (id 1) (at 44.45 83.82 0))
     (property "Footprint" "marbastlib-mx:SW_MX_1.75u" (id 2) (at 43.18 78.74 0)
       (effects (font (size 1.27 1.27)) hide)
@@
     (pin "2")
   )
-  (symbol (lib_id "marbastlib-mx:MX_SW_solder") (at 210.82 99.06 0) (unit 1)
-    (in_bom yes) (on_board yes)
-    (property "Reference" "SW61" (id 0) (at 210.82 91.44 0))
-    (property "Value" "MX_SW_solder" (id 1) (at 209.55 93.98 0))
+  (symbol (lib_id "marbastlib-mx:MX_SW_solder") (at 210.82 99.06 180) (unit 1)
+    (in_bom yes) (on_board yes)
+    (property "Reference" "SW61" (id 0) (at 210.82 106.68 0))
+    (property "Value" "MX_SW_solder" (id 1) (at 212.09 104.14 0))
     (property "Footprint" "marbastlib-mx:SW_MX_1u" (id 2) (at 210.82 99.06 0)
       (effects (font (size 1.27 1.27)) hide)
@@
     (pin "2")
   )
-  (symbol (lib_id "marbastlib-mx:MX_SW_solder") (at 241.3 58.42 0) (unit 1)
-    (in_bom yes) (on_board yes)
-    (property "Reference" "SW29" (id 0) (at 241.3 50.8 0))
-    (property "Value" "MX_SW_solder" (id 1) (at 240.03 53.34 0))
+  (symbol (lib_id "marbastlib-mx:MX_SW_solder") (at 241.3 58.42 180) (unit 1)
+    (in_bom yes) (on_board yes)
+    (property "Reference" "SW29" (id 0) (at 241.3 66.04 0))
+    (property "Value" "MX_SW_solder" (id 1) (at 242.57 63.5 0))
     (property "Footprint" "marbastlib-mx:SW_MX_1.5u" (id 2) (at 241.3 58.42 0)
       (effects (font (size 1.27 1.27)) hide)
@@
     (pin "2")
   )
-  (symbol (lib_id "marbastlib-mx:MX_SW_solder") (at 241.3 38.1 0) (unit 1)
-    (in_bom yes) (on_board yes)
-    (property "Reference" "SW15" (id 0) (at 241.3 30.48 0))
-    (property "Value" "MX_SW_solder" (id 1) (at 240.03 33.02 0))
+  (symbol (lib_id "marbastlib-mx:MX_SW_solder") (at 241.3 38.1 180) (unit 1)
+    (in_bom yes) (on_board yes)
+    (property "Reference" "SW15" (id 0) (at 241.3 45.72 0))
+    (property "Value" "MX_SW_solder" (id 1) (at 242.57 43.18 0))
     (property "Footprint" "marbastlib-mx:SW_MX_1u" (id 2) (at 241.3 38.1 0)
       (effects (font (size 1.27 1.27)) hide)
@@
     (pin "2")
   )
-  (symbol (lib_id "marbastlib-mx:MX_SW_solder") (at 182.88 119.38 180) (unit 1)
-    (in_bom yes) (on_board yes)
-    (property "Reference" "SW80" (id 0) (at 182.88 127 0))
-    (property "Value" "MX_SW_solder" (id 1) (at 184.15 124.46 0))
+  (symbol (lib_id "marbastlib-mx:MX_SW_solder") (at 182.88 119.38 0) (unit 1)
+    (in_bom yes) (on_board yes)
+    (property "Reference" "SW80" (id 0) (at 182.88 111.76 0))
+    (property "Value" "MX_SW_solder" (id 1) (at 181.61 114.3 0))
     (property "Footprint" "marbastlib-mx:SW_MX_1.25u" (id 2) (at 182.88 119.38 0)
       (effects (font (size 1.27 1.27)) hide)
@@
     (pin "2")
   )
-  (symbol (lib_id "marbastlib-mx:MX_SW_solder") (at 26.67 78.74 0) (mirror y) (unit 1)
-    (in_bom yes) (on_board yes)
-    (property "Reference" "SW31" (id 0) (at 26.67 71.12 0))
-    (property "Value" "MX_SW_solder" (id 1) (at 27.94 73.66 0))
+  (symbol (lib_id "marbastlib-mx:MX_SW_solder") (at 26.67 78.74 0) (mirror x) (unit 1)
+    (in_bom yes) (on_board yes)
+    (property "Reference" "SW31" (id 0) (at 26.67 86.36 0))
+    (property "Value" "MX_SW_solder" (id 1) (at 25.4 83.82 0))
     (property "Footprint" "marbastlib-mx:SW_MX_1.75u_stp" (id 2) (at 26.67 78.74 0)
       (effects (font (size 1.27 1.27)) hide)
@@
     (pin "2")
   )
-  (symbol (lib_id "marbastlib-mx:MX_SW_solder") (at 247.65 52.07 0) (unit 1)
-    (in_bom yes) (on_board yes)
-    (property "Reference" "SW30" (id 0) (at 259.08 48.26 0))
-    (property "Value" "MX_SW_solder" (id 1) (at 257.81 50.8 0))
+  (symbol (lib_id "marbastlib-mx:MX_SW_solder") (at 247.65 52.07 180) (unit 1)
+    (in_bom yes) (on_board yes)
+    (property "Reference" "SW30" (id 0) (at 236.22 55.88 0))
+    (property "Value" "MX_SW_solder" (id 1) (at 237.49 53.34 0))
     (property "Footprint" "marbastlib-mx:SW_MX_1u" (id 2) (at 247.65 52.07 0)
       (effects (font (size 1.27 1.27)) hide)
@@
     (pin "2")
   )
-  (symbol (lib_id "marbastlib-mx:MX_SW_solder") (at 43.18 99.06 0) (unit 1)
-    (in_bom yes) (on_board yes)
-    (property "Reference" "SW48" (id 0) (at 43.18 91.44 0))
-    (property "Value" "MX_SW_solder" (id 1) (at 41.91 93.98 0))
+  (symbol (lib_id "marbastlib-mx:MX_SW_solder") (at 43.18 99.06 180) (unit 1)
+    (in_bom yes) (on_board yes)
+    (property "Reference" "SW48" (id 0) (at 43.18 106.68 0))
+    (property "Value" "MX_SW_solder" (id 1) (at 44.45 104.14 0))
     (property "Footprint" "marbastlib-mx:SW_MX_1u" (id 2) (at 43.18 99.06 0)
       (effects (font (size 1.27 1.27)) hide)
@@
     (pin "2")
   )
-  (symbol (lib_id "marbastlib-mx:MX_SW_solder") (at 27.94 99.06 0) (mirror y) (unit 1)
-    (in_bom yes) (on_board yes)
-    (property "Reference" "SW47" (id 0) (at 27.94 91.44 0))
-    (property "Value" "MX_SW_solder" (id 1) (at 29.21 93.98 0))
+  (symbol (lib_id "marbastlib-mx:MX_SW_solder") (at 27.94 99.06 0) (mirror x) (unit 1)
+    (in_bom yes) (on_board yes)
+    (property "Reference" "SW47" (id 0) (at 27.94 106.68 0))
+    (property "Value" "MX_SW_solder" (id 1) (at 26.67 104.14 0))
     (property "Footprint" "marbastlib-mx:SW_MX_1.25u" (id 2) (at 27.94 99.06 0)
       (effects (font (size 1.27 1.27)) hide)
@@
     (pin "2")
   )
-  (symbol (lib_id "marbastlib-mx:MX_SW_solder") (at 217.17 92.71 0) (unit 1)
-    (in_bom yes) (on_board yes)
-    (property "Reference" "SW60" (id 0) (at 227.33 90.17 0))
-    (property "Value" "MX_SW_solder" (id 1) (at 226.06 92.71 0))
+  (symbol (lib_id "marbastlib-mx:MX_SW_solder") (at 217.17 92.71 180) (unit 1)
+    (in_bom yes) (on_board yes)
+    (property "Reference" "SW60" (id 0) (at 207.01 95.25 0))
+    (property "Value" "MX_SW_solder" (id 1) (at 208.28 92.71 0))
     (property "Footprint" "marbastlib-mx:SW_MX_1.75u" (id 2) (at 217.17 92.71 0)
       (effects (font (size 1.27 1.27)) hide)
@@
     (pin "2")
   )
-  (symbol (lib_id "marbastlib-mx:MX_SW_solder") (at 241.3 139.7 0) (mirror x) (unit 1)
-    (in_bom yes) (on_board yes)
-    (property "Reference" "SW88" (id 0) (at 241.3 147.32 0))
-    (property "Value" "MX_SW_solder" (id 1) (at 240.03 144.78 0))
+  (symbol (lib_id "marbastlib-mx:MX_SW_solder") (at 241.3 139.7 0) (mirror y) (unit 1)
+    (in_bom yes) (on_board yes)
+    (property "Reference" "SW88" (id 0) (at 241.3 132.08 0))
+    (property "Value" "MX_SW_solder" (id 1) (at 242.57 134.62 0))
     (property "Footprint" "marbastlib-mx:SW_MX_1.5u" (id 2) (at 241.3 139.7 0)
       (effects (font (size 1.27 1.27)) hide)
@@
     (pin "2")
   )
-  (symbol (lib_id "marbastlib-mx:MX_SW_solder") (at 241.3 119.38 0) (unit 1)
-    (in_bom yes) (on_board yes)
-    (property "Reference" "SW87" (id 0) (at 241.3 111.76 0))
-    (property "Value" "MX_SW_solder" (id 1) (at 240.03 114.3 0))
+  (symbol (lib_id "marbastlib-mx:MX_SW_solder") (at 241.3 119.38 180) (unit 1)
+    (in_bom yes) (on_board yes)
+    (property "Reference" "SW87" (id 0) (at 241.3 127 0))
+    (property "Value" "MX_SW_solder" (id 1) (at 242.57 124.46 0))
     (property "Footprint" "marbastlib-mx:SW_MX_1.25u" (id 2) (at 241.3 119.38 0)
       (effects (font (size 1.27 1.27)) hide)
@@
     (pin "2")
   )
-  (symbol (lib_id "marbastlib-mx:MX_SW_solder") (at 241.3 99.06 0) (unit 1)
-    (in_bom yes) (on_board yes)
-    (property "Reference" "SW62" (id 0) (at 241.3 91.44 0))
-    (property "Value" "MX_SW_solder" (id 1) (at 240.03 93.98 0))
+  (symbol (lib_id "marbastlib-mx:MX_SW_solder") (at 241.3 99.06 180) (unit 1)
+    (in_bom yes) (on_board yes)
+    (property "Reference" "SW62" (id 0) (at 241.3 106.68 0))
+    (property "Value" "MX_SW_solder" (id 1) (at 242.57 104.14 0))
     (property "Footprint" "marbastlib-mx:SW_MX_1u" (id 2) (at 241.3 99.06 0)
       (effects (font (size 1.27 1.27)) hide)
@@
     (pin "2")
   )
-  (symbol (lib_id "marbastlib-mx:MX_SW_solder") (at 247.65 29.21 0) (unit 1)
-    (in_bom yes) (on_board yes)
-    (property "Reference" "SW14" (id 0) (at 247.65 21.59 0))
-    (property "Value" "MX_SW_solder" (id 1) (at 246.38 24.13 0))
+  (symbol (lib_id "marbastlib-mx:MX_SW_solder") (at 247.65 29.21 180) (unit 1)
+    (in_bom yes) (on_board yes)
+    (property "Reference" "SW14" (id 0) (at 247.65 36.83 0))
+    (property "Value" "MX_SW_solder" (id 1) (at 248.92 34.29 0))
     (property "Footprint" "marbastlib-mx:SW_MX_1u" (id 2) (at 247.65 29.21 0)
       (effects (font (size 1.27 1.27)) hide)
@@
     (pin "2")
   )
-  (symbol (lib_id "marbastlib-mx:MX_SW_solder") (at 210.82 58.42 0) (unit 1)
-    (in_bom yes) (on_board yes)
-    (property "Reference" "SW28" (id 0) (at 210.82 50.8 0))
-    (property "Value" "MX_SW_solder" (id 1) (at 209.55 53.34 0))
+  (symbol (lib_id "marbastlib-mx:MX_SW_solder") (at 210.82 58.42 180) (unit 1)
+    (in_bom yes) (on_board yes)
+    (property "Reference" "SW28" (id 0) (at 210.82 66.04 0))
+    (property "Value" "MX_SW_solder" (id 1) (at 212.09 63.5 0))
     (property "Footprint" "marbastlib-mx:SW_MX_1u" (id 2) (at 210.82 58.42 0)
       (effects (font (size 1.27 1.27)) hide)

Commit message: preliminary SMD component placements
Connections:
- net COL00: now also SW16.2; no longer SW16.1
- net at D16.2 (A): now also SW16.1; no longer SW16.2
Other:
- moved on the sheet: SW16
Changed lines of the file:
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@@
     (pin "2")
   )
-  (symbol (lib_id "marbastlib-mx:MX_SW_solder") (at 43.18 58.42 0) (unit 1)
+  (symbol (lib_id "marbastlib-mx:MX_SW_solder") (at 43.18 58.42 180) (unit 1)
     (in_bom yes) (on_board yes)
-    (property "Reference" "SW16" (id 0) (at 43.18 50.8 0))
-    (property "Value" "MX_SW_solder" (id 1) (at 41.91 53.34 0))
+    (property "Reference" "SW16" (id 0) (at 43.18 66.04 0))
+    (property "Value" "MX_SW_solder" (id 1) (at 44.45 63.5 0))
     (property "Footprint" "marbastlib-mx:SW_MX_1.5u" (id 2) (at 43.18 58.42 0)
       (effects (font (size 1.27 1.27)) hide)

Commit message: clean up
Parts:
- renumbered D16 to D15, D17 to D16, D18 to D17, D19 to D18, D20 to D19, D21 to D20, D22 to D21, D23 to D22, D24 to D23, D25 to D24, D26 to D25, D27 to D26, D28 to D27, D29 to D28, D32 to D29, D33 to D30, D34 to D31, D35 to D32, D36 to D33, D37 to D34, D38 to D35, D39 to D36, D40 to D37, D41 to D38, D42 to D39, D43 to D40, D44 to D41, D46 to D42, D48 to D43, D49 to D44, D50 to D45, D51 to D46, D52 to D47, D53 to D48, D54 to D49, D55 to D50, D56 to D51, D57 to D52, D58 to D53, D59 to D54, D60 to D55, D62 to D56, D63 to D57, D65 to D58, D68 to D59, D71 to D60, D73 to D61, D77 to D62, D80 to D63, D81 to D64, D84 to D65, D87 to D66

Commit message: o ring mounting cutouts
Parts:
- removed SW76: MX_SW_solder, marbastlib-mx:SW_MX_1.25u, symbol marbastlib-mx:MX_SW_solder
- removed SW79: MX_SW_solder, marbastlib-mx:SW_MX_1u, symbol marbastlib-mx:MX_SW_solder
- renumbered SW77 to SW76, SW78 to SW77, SW80 to SW78, SW81 to SW79, SW82 to SW80, SW83 to SW81, SW84 to SW82, SW85 to SW83, SW86 to SW84, SW87 to SW85, SW88 to SW86
Connections:
- net COL08: now also SW77.1; no longer SW77.2
- net at D62.2 (A), SW76.2: now also SW77.2; no longer SW77.1
Changed lines of the file:
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@@
   (junction (at 185.42 88.9) (diameter 0) (color 0 0 0 0)
   )
-  (junction (at 119.38 160.02) (diameter 0) (color 0 0 0 0)
-  )
   (junction (at 203.2 69.85) (diameter 0) (color 0 0 0 0)
   )
@@
   (junction (at 129.54 68.58) (diameter 0) (color 0 0 0 0)
   )
-  (junction (at 160.02 137.16) (diameter 0) (color 0 0 0 0)
-  )
   (junction (at 213.36 48.26) (diameter 0) (color 0 0 0 0)
   )
@@
   (junction (at 243.84 121.92) (diameter 0) (color 0 0 0 0)
   )
-  (junction (at 147.32 142.24) (diameter 0) (color 0 0 0 0)
-  )
   (junction (at 213.36 81.28) (diameter 0) (color 0 0 0 0)
   )
@@
   (junction (at 201.93 137.16) (diameter 0) (color 0 0 0 0)
   )
-  (junction (at 137.16 154.94) (diameter 0) (color 0 0 0 0)
-  )
   (junction (at 233.68 26.67) (diameter 0) (color 0 0 0 0)
   )
@@
     (stroke (width 0) (type default) (color 0 0 0 0))
   )
-  (wire (pts (xy 137.16 154.94) (xy 137.16 167.64))
-    (stroke (width 0) (type default) (color 0 0 0 0))
-  )
   (wire (pts (xy 185.42 48.26) (xy 199.39 48.26))
     (stroke (width 0) (type default) (color 0 0 0 0))
@@
     (stroke (width 0) (type default) (color 0 0 0 0))
   )
-  (wire (pts (xy 119.38 172.72) (xy 119.38 160.02))
-    (stroke (width 0) (type default) (color 0 0 0 0))
-  )
   (wire (pts (xy 63.5 96.52) (xy 68.58 96.52))
     (stroke (width 0) (type default) (color 0 0 0 0))
@@
     (stroke (width 0) (type default) (color 0 0 0 0))
   )
-  (wire (pts (xy 160.02 154.94) (xy 160.02 137.16))
-    (stroke (width 0) (type default) (color 0 0 0 0))
-  )
   (wire (pts (xy 157.48 88.9) (xy 171.45 88.9))
     (stroke (width 0) (type default) (color 0 0 0 0))
@@
     (stroke (width 0) (type default) (color 0 0 0 0))
   )
-  (wire (pts (xy 132.08 172.72) (xy 119.38 172.72))
-    (stroke (width 0) (type default) (color 0 0 0 0))
-  )
   (wire (pts (xy 143.51 109.22) (xy 157.48 109.22))
     (stroke (width 0) (type default) (color 0 0 0 0))
@@
     (stroke (width 0) (type default) (color 0 0 0 0))
   )
-  (wire (pts (xy 147.32 160.02) (xy 147.32 142.24))
-    (stroke (width 0) (type default) (color 0 0 0 0))
-  )
   (wire (pts (xy 161.29 76.2) (xy 166.37 76.2))
     (stroke (width 0) (type default) (color 0 0 0 0))
@@
     (stroke (width 0) (type default) (color 0 0 0 0))
   )
-  (wire (pts (xy 154.94 160.02) (xy 147.32 160.02))
-    (stroke (width 0) (type default) (color 0 0 0 0))
-  )
   (wire (pts (xy 199.39 129.54) (xy 213.36 129.54))
     (stroke (width 0) (type default) (color 0 0 0 0))
@@
   (symbol (lib_id "marbastlib-mx:MX_SW_solder") (at 196.85 119.38 0) (unit 1)
     (in_bom yes) (on_board yes)
-    (property "Reference" "SW81" (id 0) (at 196.85 111.76 0))
+    (property "Reference" "SW79" (id 0) (at 196.85 111.76 0))
     (property "Value" "MX_SW_solder" (id 1) (at 195.58 114.3 0))
     (property "Footprint" "marbastlib-mx:SW_MX_1.25u" (id 2) (at 196.85 119.38 0)
@@
   (symbol (lib_id "marbastlib-mx:MX_SW_solder") (at 199.39 157.48 0) (mirror x) (unit 1)
     (in_bom yes) (on_board yes)
-    (property "Reference" "SW83" (id 0) (at 199.39 165.1 0))
+    (property "Reference" "SW81" (id 0) (at 199.39 165.1 0))
     (property "Value" "MX_SW_solder" (id 1) (at 198.12 162.56 0))
     (property "Footprint" "marbastlib-mx:SW_MX_1.25u" (id 2) (at 199.39 157.48 0)
@@
   (symbol (lib_id "marbastlib-mx:MX_SW_solder") (at 210.82 139.7 0) (mirror x) (unit 1)
     (in_bom yes) (on_board yes)
-    (property "Reference" "SW85" (id 0) (at 210.82 147.32 0))
+    (property "Reference" "SW83" (id 0) (at 210.82 147.32 0))
     (property "Value" "MX_SW_solder" (id 1) (at 209.55 144.78 0))
     (property "Footprint" "marbastlib-mx:SW_MX_1u" (id 2) (at 210.82 139.7 0)
@@
     (pin "2")
   )
-  (symbol (lib_id "marbastlib-mx:MX_SW_solder") (at 157.48 157.48 0) (mirror x) (unit 1)
-    (in_bom yes) (on_board yes)
-    (property "Reference" "SW79" (id 0) (at 157.48 165.1 0))
-    (property "Value" "MX_SW_solder" (id 1) (at 156.21 162.56 0))
-    (property "Footprint" "marbastlib-mx:SW_MX_1u" (id 2) (at 157.48 157.48 0)
-      (effects (font (size 1.27 1.27)) hide)
-    )
-    (property "Datasheet" "~" (id 3) (at 157.48 157.48 0)
-      (effects (font (size 1.27 1.27)) hide)
-    )
-    (pin "1")
-    (pin "2")
-  )
   (symbol (lib_id "marbastlib-mx:MX_SW_solder") (at 71.12 119.38 0) (unit 1)
     (in_bom yes) (on_board yes)
@@
   (symbol (lib_id "marbastlib-mx:MX_SW_solder") (at 210.82 119.38 0) (unit 1)
     (in_bom yes) (on_board yes)
-    (property "Reference" "SW84" (id 0) (at 210.82 111.76 0))
+    (property "Reference" "SW82" (id 0) (at 210.82 111.76 0))
     (property "Value" "MX_SW_solder" (id 1) (at 209.55 114.3 0))
     (property "Footprint" "marbastlib-mx:SW_MX_1.25u" (id 2) (at 210.82 119.38 0)
@@
   (symbol (lib_id "marbastlib-mx:MX_SW_solder") (at 154.94 119.38 0) (unit 1)
     (in_bom yes) (on_board yes)
-    (property "Reference" "SW77" (id 0) (at 154.94 111.76 0))
+    (property "Reference" "SW76" (id 0) (at 154.94 111.76 0))
     (property "Value" "MX_SW_solder" (id 1) (at 153.67 114.3 0))
     (property "Footprint" "marbastlib-mx:SW_MX_1u" (id 2) (at 154.94 119.38 0)
@@
     (pin "2")
   )
-  (symbol (lib_id "marbastlib-mx:MX_SW_solder") (at 134.62 170.18 0) (mirror x) (unit 1)
-    (in_bom yes) (on_board yes)
-    (property "Reference" "SW76" (id 0) (at 134.62 177.8 0))
-    (property "Value" "MX_SW_solder" (id 1) (at 133.35 175.26 0))
-    (property "Footprint" "marbastlib-mx:SW_MX_1.25u" (id 2) (at 134.62 170.18 0)
-      (effects (font (size 1.27 1.27)) hide)
-    )
-    (property "Datasheet" "~" (id 3) (at 134.62 170.18 0)
-      (effects (font (size 1.27 1.27)) hide)
-    )
-    (pin "1")
-    (pin "2")
-  )
   (symbol (lib_id "Device:D_Small") (at 243.84 124.46 90) (unit 1)
     (in_bom yes) (on_board yes)
@@
   (symbol (lib_id "marbastlib-mx:MX_SW_solder") (at 213.36 157.48 0) (mirror x) (unit 1)
     (in_bom yes) (on_board yes)
-    (property "Reference" "SW86" (id 0) (at 213.36 165.1 0))
+    (property "Reference" "SW84" (id 0) (at 213.36 165.1 0))
     (property "Value" "MX_SW_solder" (id 1) (at 212.09 162.56 0))
     (property "Footprint" "marbastlib-mx:SW_MX_1.25u" (id 2) (at 213.36 157.48 0)
@@
   (symbol (lib_id "marbastlib-mx:MX_SW_solder") (at 182.88 119.38 0) (unit 1)
     (in_bom yes) (on_board yes)
-    (property "Reference" "SW80" (id 0) (at 182.88 111.76 0))
+    (property "Reference" "SW78" (id 0) (at 182.88 111.76 0))
     (property "Value" "MX_SW_solder" (id 1) (at 181.61 114.3 0))
     (property "Footprint" "marbastlib-mx:SW_MX_1.25u" (id 2) (at 182.88 119.38 0)
@@
   (symbol (lib_id "marbastlib-mx:MX_SW_solder") (at 241.3 139.7 0) (mirror y) (unit 1)
     (in_bom yes) (on_board yes)
-    (property "Reference" "SW88" (id 0) (at 241.3 132.08 0))
+    (property "Reference" "SW86" (id 0) (at 241.3 132.08 0))
     (property "Value" "MX_SW_solder" (id 1) (at 242.57 134.62 0))
     (property "Footprint" "marbastlib-mx:SW_MX_1.5u" (id 2) (at 241.3 139.7 0)
@@
     (pin "2")
   )
-  (symbol (lib_id "marbastlib-mx:MX_SW_solder") (at 154.94 139.7 0) (mirror y) (unit 1)
+  (symbol (lib_id "marbastlib-mx:MX_SW_solder") (at 154.94 139.7 0) (mirror x) (unit 1)
     (in_bom yes) (on_board yes)
-    (property "Reference" "SW78" (id 0) (at 154.94 132.08 0))
-    (property "Value" "MX_SW_solder" (id 1) (at 156.21 134.62 0))
+    (property "Reference" "SW77" (id 0) (at 154.94 135.89 0))
+    (property "Value" "MX_SW_solder" (id 1) (at 153.67 133.35 0))
     (property "Footprint" "marbastlib-mx:SW_MX_1u" (id 2) (at 154.94 139.7 0)
       (effects (font (size 1.27 1.27)) hide)
@@
   (symbol (lib_id "marbastlib-mx:MX_SW_solder") (at 241.3 119.38 180) (unit 1)
     (in_bom yes) (on_board yes)
-    (property "Reference" "SW87" (id 0) (at 245.11 118.11 0))
+    (property "Reference" "SW85" (id 0) (at 245.11 118.11 0))
     (property "Value" "MX_SW_solder" (id 1) (at 246.38 115.57 0))
     (property "Footprint" "marbastlib-mx:SW_MX_1.25u" (id 2) (at 241.3 119.38 0)
@@
   (symbol (lib_id "marbastlib-mx:MX_SW_solder") (at 196.85 139.7 0) (mirror x) (unit 1)
     (in_bom yes) (on_board yes)
-    (property "Reference" "SW82" (id 0) (at 196.85 147.32 0))
+    (property "Reference" "SW80" (id 0) (at 196.85 147.32 0))
     (property "Value" "MX_SW_solder" (id 1) (at 195.58 144.78 0))
     (property "Footprint" "marbastlib-mx:SW_MX_1.5u" (id 2) (at 196.85 139.7 0)

Commit message: swap bulk cap & reroute debug
Connections:
- net COL12: now also SW28.1; no longer SW28.2
- net at D27.2 (A): now also SW28.2; no longer SW28.1
Other:
- moved on the sheet: SW28
Changed lines of the file:
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@@
     (pin "2")
   )
-  (symbol (lib_id "marbastlib-mx:MX_SW_solder") (at 210.82 58.42 180) (unit 1)
+  (symbol (lib_id "marbastlib-mx:MX_SW_solder") (at 210.82 58.42 0) (unit 1)
     (in_bom yes) (on_board yes)
-    (property "Reference" "SW28" (id 0) (at 217.17 58.42 0))
-    (property "Value" "MX_SW_solder" (id 1) (at 218.44 55.88 0))
+    (property "Reference" "SW28" (id 0) (at 214.63 50.8 0))
+    (property "Value" "MX_SW_solder" (id 1) (at 213.36 53.34 0))
     (property "Footprint" "marbastlib-mx:SW_MX_1u" (id 2) (at 210.82 58.42 0)
       (effects (font (size 1.27 1.27)) hide)
