File: ice60.kicad_sch (KiCad schematic)
At the start: 34 parts, among them J1 SWD, J2 JST SH 4-pin, SW0 SW_Push, U1 RP2040, U2 W25Q128JVS, U3 XC6206PxxxMR, U4 SRV05-4, Y1 12MHz

Commit message: add part numbers for BOM
Parts:
- D67, D68: now left out of the parts list
- F1: LCSC (none) -> C135342
- J2: LCSC (none) -> C160404
- R2, R3: value 22R -> 27R
- R6: value 470 -> 470R; LCSC (none) -> C25117
- U1: LCSC (none) -> C2040
- U3: LCSC (none) -> C5446
- U4: LCSC (none) -> C85364
Changed lines of the file:
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@@
   (title_block
     (title "ice60")
-    (date "2022-12-27")
+    (date "2023-01-04")
     (company "chill")
     (comment 1 "© 2022 chillKB")
@@
   )
   (symbol (lib_id "Device:LED") (at 227.33 104.14 270) (mirror x) (unit 1)
-    (in_bom yes) (on_board yes)
+    (in_bom no) (on_board yes)
     (property "Reference" "D67" (id 0) (at 219.71 104.14 90)
       (effects (font (size 1.27 1.27)) (justify left))
@@
     )
     (property "Datasheet" "http://www.onsemi.com/pub/Collateral/SRV05-4-D.PDF" (id 3) (at 240.03 35.56 0)
+      (effects (font (size 1.27 1.27)) hide)
+    )
+    (property "LCSC" "C85364" (id 4) (at 240.03 35.56 0)
       (effects (font (size 1.27 1.27)) hide)
     )
@@
     (in_bom yes) (on_board yes)
     (property "Reference" "R3" (id 0) (at 29.21 45.72 90))
-    (property "Value" "22R" (id 1) (at 36.83 45.72 90))
+    (property "Value" "27R" (id 1) (at 36.83 45.72 90))
     (property "Footprint" "Resistor_SMD:R_0603_1608Metric" (id 2) (at 33.02 46.99 0)
       (effects (font (size 1.27 1.27)) hide)
@@
     )
     (property "Datasheet" "~" (id 3) (at 209.55 69.85 0)
+      (effects (font (size 1.27 1.27)) hide)
+    )
+    (property "LCSC" "C160404" (id 4) (at 209.55 69.85 0)
       (effects (font (size 1.27 1.27)) hide)
     )
@@
       (effects (font (size 1.27 1.27)) hide)
     )
+    (property "LCSC" "C5446" (id 4) (at 195.58 38.1 0)
+      (effects (font (size 1.27 1.27)) hide)
+    )
     (pin "1")
     (pin "2")
@@
     (in_bom yes) (on_board yes)
     (property "Reference" "R2" (id 0) (at 29.21 43.18 90))
-    (property "Value" "22R" (id 1) (at 36.83 43.18 90))
+    (property "Value" "27R" (id 1) (at 36.83 43.18 90))
     (property "Footprint" "Resistor_SMD:R_0603_1608Metric" (id 2) (at 33.02 44.45 0)
       (effects (font (size 1.27 1.27)) hide)
@@
   )
   (symbol (lib_id "Device:LED") (at 232.41 104.14 90) (unit 1)
-    (in_bom yes) (on_board yes) (fields_autoplaced)
+    (in_bom no) (on_board yes) (fields_autoplaced)
     (property "Reference" "D68" (id 0) (at 236.22 104.4574 90)
       (effects (font (size 1.27 1.27)) (justify right))
@@
       (effects (font (size 1.27 1.27)) (justify left))
     )
-    (property "Value" "470" (id 1) (at 232.41 99.0599 0)
+    (property "Value" "470R" (id 1) (at 232.41 99.0599 0)
       (effects (font (size 1.27 1.27)) (justify left))
     )
@@
     )
     (property "Datasheet" "~" (id 3) (at 229.87 97.79 0)
+      (effects (font (size 1.27 1.27)) hide)
+    )
+    (property "LCSC" "C25117" (id 4) (at 229.87 97.79 0)
       (effects (font (size 1.27 1.27)) hide)
     )
@@
       (effects (font (size 1.27 1.27)) hide)
     )
+    (property "LCSC" "C135342" (id 4) (at 228.6 67.31 0)
+      (effects (font (size 1.27 1.27)) hide)
+    )
     (pin "1")
     (pin "2")
@@
     (property "Datasheet" "https://datasheets.raspberrypi.com/rp2040/rp2040-datasheet.pdf" (id 3) (at 43.18 13.97 0)
       (effects (font (size 1.27 1.27)) (justify left bottom) hide)
+    )
+    (property "LCSC" "C2040" (id 4) (at 63.5 76.2 0)
+      (effects (font (size 1.27 1.27)) hide)
     )
     (pin "1")
@@
     )
     (path "/bd723373-d5f4-49eb-b3bb-9d45633445a1"
-      (reference "R2") (unit 1) (value "22R") (footprint "Resistor_SMD:R_0603_1608Metric")
+      (reference "R2") (unit 1) (value "27R") (footprint "Resistor_SMD:R_0603_1608Metric")
     )
     (path "/94851e3a-d156-41bd-8091-39411b3366f5"
-      (reference "R3") (unit 1) (value "22R") (footprint "Resistor_SMD:R_0603_1608Metric")
+      (reference "R3") (unit 1) (value "27R") (footprint "Resistor_SMD:R_0603_1608Metric")
     )
     (path "/80a1f407-77cc-4d9d-91be-6deef95b28bc"
@@
     )
     (path "/f4dc9ca1-a46b-480b-8045-0daec62f2914"
-      (reference "R6") (unit 1) (value "470") (footprint "Resistor_SMD:R_0402_1005Metric")
+      (reference "R6") (unit 1) (value "470R") (footprint "Resistor_SMD:R_0402_1005Metric")
     )
     (path "/99b63952-0e82-445f-a871-af9a28c1c443"

Commit message: update to kicad 7, many small changes
Parts:
- F1: LCSC C135342 -> C70076
- U2: LCSC C131025 -> C97521
